Commit message: basic control plugin built

File: viman_visualize/urdf/viman.xacro (robot description, xacro)
@@ -43,5 +43,5 @@
 			</collision>
         </link>
-        <joint name="propeller_${id}_joint" type="continuous">
+        <joint name="propeller_${id}_joint" type="fixed">
             <parent link="base_link"/>
             <child link="propeller_${id}"/>
@@ -99,3 +99,32 @@
   <xacro:propeller_link id="3" com="-2.7756E-17 -0.00027271 0" xyz="0.085003 0.084703 0.0335" rpy="1.5708 0 1.1739"/>
   <xacro:propeller_link id="4" com="2.7756E-17 -0.00027271 2.7756E-17" xyz="-0.084703 0.085003 0.0335" rpy="1.5708 0 2.5345"/>
+  <gazebo>
+    <plugin name='uav_viman' filename='libplugin_viman_ctrl.so'>
+        <bodyName>base_link</bodyName>
+        <imuTopic>/viman/imu</imuTopic>
+        <rollpitchProportionalGain>10.0</rollpitchProportionalGain>
+        <rollpitchDifferentialGain>5.0</rollpitchDifferentialGain>
+        <rollpitchLimit>0.5</rollpitchLimit>
+        <yawProportionalGain>2.0</yawProportionalGain>
+        <yawDifferentialGain>1.0</yawDifferentialGain>
+        <yawLimit>1.5</yawLimit>
+        <velocityXYProportionalGain>5.0</velocityXYProportionalGain>
+        <velocityXYDifferentialGain>2.3</velocityXYDifferentialGain>
+        <velocityXYLimit>2</velocityXYLimit>
+        <velocityZProportionalGain>5.0</velocityZProportionalGain>
+        <velocityZDifferentialGain>1.0</velocityZDifferentialGain>
+        <velocityZLimit>-1</velocityZLimit>
+        <positionXYProportionalGain>1.1</positionXYProportionalGain>
+        <positionXYDifferentialGain>0.0</positionXYDifferentialGain>
+        <positionXYIntegralGain>0.0</positionXYIntegralGain>
+        <positionXYLimit>5</positionXYLimit>
+        <positionZProportionalGain>1.0</positionZProportionalGain>
+        <positionZDifferentialGain>0.2</positionZDifferentialGain>
+        <positionZLimit>-1</positionZLimit>
+        <maxForce>30</maxForce>
+        <motionSmallNoise>0.05</motionSmallNoise>
+        <motionDriftNoise>0.03</motionDriftNoise>
+        <motionDriftNoiseTime>5.0</motionDriftNoiseTime>
+    </plugin>
+  </gazebo>
 </robot>

Commit message: added key-ctrl and basic altimeter

File: viman_visualize/urdf/viman.xacro (robot description, xacro)
@@ -56,8 +56,8 @@
     <inertial>
       <origin
-        xyz="-2.0447E-05 0.019934 -2.776E-05"
+        xyz="0 0 0"
         rpy="0 0 0" />
       <mass
-        value="0.2066" />
+        value="0.6" />
       <inertia
         ixx="3.294E-05"
@@ -100,5 +100,5 @@
   <xacro:propeller_link id="4" com="2.7756E-17 -0.00027271 2.7756E-17" xyz="-0.084703 0.085003 0.0335" rpy="1.5708 0 2.5345"/>
   <gazebo>
-    <plugin name='uav_viman' filename='libplugin_viman_ctrl.so'>
+    <plugin name='viman_flight' filename='libplugin_viman_flight.so'>
         <bodyName>base_link</bodyName>
         <imuTopic>/viman/imu</imuTopic>
@@ -128,3 +128,108 @@
     </plugin>
   </gazebo>
+  <xacro:property name="cam_origin_offset" value="0 -0.03 0.01"/>
+  <xacro:property name="camera_dimensions" value="0.01 0.01 0.01"/>
+  <xacro:property name="altimeter_origin_offset" value="0 0 0.1"/>
+  <xacro:property name="altimeter_dimensions" value="0.005 0.005 0.005"/>
+  <link name="camera">
+    <collision>
+      <origin xyz="0 0 0" rpy="0 0 0"/>
+      <geometry>
+		<box size="${camera_dimensions}"/>
+      </geometry>
+    </collision>
+    <visual>
+      <origin xyz="0 0 0" rpy="0 0 0"/>
+      <geometry>
+    <box size="${camera_dimensions}"/>
+      </geometry>
+      <material name="red"/>
+    </visual>
+    <inertial>
+      <mass value="1e-5" />
+      <origin xyz="0 0 0" rpy="0 0 0"/>
+      <inertia ixx="1e-6" ixy="0" ixz="0" iyy="1e-6" iyz="0" izz="1e-6" />
+    </inertial>
+  </link>
+  <joint name="camera_joint" type="fixed">
+    <origin xyz="${cam_origin_offset}" rpy="0 0 -1.5708"/>
+    <parent link="base_link"/>
+    <child link="camera"/>
+  </joint>
+  <!-- Camera: Plugin -->
+  <gazebo reference="camera">
+	<material>Gazebo/Red</material>
+    <sensor type="camera" name="viman_frnt_cam">
+      <update_rate>30.0</update_rate>
+      <camera name="viman_frnt_cam">
+        <horizontal_fov>1.3962634</horizontal_fov>
+        <image>
+          <width>800</width>
+          <height>800</height>
+          <format>R8G8B8</format>
+        </image>
+        <clip>
+          <near>0.02</near>
+          <far>300</far>
+        </clip>
+        <noise>
+          <type>gaussian</type>
+          <!-- Noise is sampled independently per pixel on each frame.
+               That pixel's noise value is added to each of its color
+               channels, which at that point lie in the range [0,1]. -->
+          <mean>0.0</mean>
+          <stddev>0.007</stddev>
+        </noise>
+      </camera>
+      <plugin name="camera_controller" filename="libgazebo_ros_camera.so">
+        <alwaysOn>true</alwaysOn>
+        <updateRate>0.0</updateRate>
+        <cameraName>viman_frnt_cam</cameraName>
+        <imageTopicName>viman_frnt_camera_out</imageTopicName>
+        <cameraInfoTopicName>viman_frnt_cam_info</cameraInfoTopicName>
+        <frameName>camera_link</frameName>
+        <hackBaseline>0.07</hackBaseline>
+        <distortionK1>0.0</distortionK1>
+        <distortionK2>0.0</distortionK2>
+        <distortionK3>0.0</distortionK3>
+        <distortionT1>0.0</distortionT1>
+        <distortionT2>0.0</distortionT2>
+      </plugin>
+    </sensor>
+  </gazebo>
+   <link name="altimeter">
+    <collision>
+      <origin xyz="0 0 0" rpy="0 0 0"/>
+      <geometry>
+		<box size="${altimeter_dimensions}"/>
+      </geometry>
+    </collision>
+    <visual>
+      <origin xyz="0 0 0" rpy="0 0 0"/>
+      <geometry>
+    <box size="${altimeter_dimensions}"/>
+      </geometry>
+      <material name="blue"/>
+    </visual>
+    <inertial>
+      <mass value="1e-5" />
+      <origin xyz="0 0 0" rpy="0 0 0"/>
+      <inertia ixx="1e-6" ixy="0" ixz="0" iyy="1e-6" iyz="0" izz="1e-6" />
+    </inertial>
+  </link>
+  <joint name="altimeter_joint" type="fixed">
+    <origin xyz="${altimeter_origin_offset}" rpy="0 0 0"/>
+    <parent link="base_link"/>
+    <child link="altimeter"/>
+  </joint>
+  <gazebo>
+	  <material>Gazebo/Blue</material>
+	  <plugin name='altimeter_plugin' filename='libplugin_altimeter.so'>
+		<bodyName>altimeter</bodyName>
+		<robotNamespace>/viman</robotNamespace>
+		<frameId>altimeter</frameId>
+		<altimeterTopicName>/height</altimeterTopicName>
+		<elevation>0</elevation>
+	  </plugin>
+  </gazebo>
 </robot>

Commit message: added altimeter plugin

File: viman_visualize/urdf/viman.xacro (robot description, xacro)
@@ -1,4 +1,9 @@
 <?xml version="1.0" encoding="utf-8"?>
 <robot name="viman" xmlns:xacro="http://www.ros.org/wiki/xacro">
+  <!-- Sensor properties -->
+  <xacro:property name="cam_origin_offset" value="0 -0.03 0.01"/>
+  <xacro:property name="camera_dimensions" value="0.01 0.01 0.01"/>
+  <xacro:property name="altimeter_origin_offset" value="0 0 0.015"/>
+  <xacro:property name="altimeter_dimensions" value="0.005 0.005 0.002"/>
   <!-- Macro to define propeller links -->
   <!-- Input parameters: propeller ID, pose of the joint, xyz of CoM -->
@@ -99,4 +104,5 @@
   <xacro:propeller_link id="3" com="-2.7756E-17 -0.00027271 0" xyz="0.085003 0.084703 0.0335" rpy="1.5708 0 1.1739"/>
   <xacro:propeller_link id="4" com="2.7756E-17 -0.00027271 2.7756E-17" xyz="-0.084703 0.085003 0.0335" rpy="1.5708 0 2.5345"/>
+  <!-- Flight plugin -->
   <gazebo>
     <plugin name='viman_flight' filename='libplugin_viman_flight.so'>
@@ -128,8 +134,4 @@
     </plugin>
   </gazebo>
-  <xacro:property name="cam_origin_offset" value="0 -0.03 0.01"/>
-  <xacro:property name="camera_dimensions" value="0.01 0.01 0.01"/>
-  <xacro:property name="altimeter_origin_offset" value="0 0 0.1"/>
-  <xacro:property name="altimeter_dimensions" value="0.005 0.005 0.005"/>
   <link name="camera">
     <collision>
@@ -198,5 +200,5 @@
     </sensor>
   </gazebo>
-   <link name="altimeter">
+  <link name="altimeter">
     <collision>
       <origin xyz="0 0 0" rpy="0 0 0"/>
@@ -223,12 +225,14 @@
     <child link="altimeter"/>
   </joint>
+  <gazebo reference="altimeter">
+	<material>Gazebo/SkyBlue</material>
+  </gazebo>
+  <!-- Altimeter plugin -->
   <gazebo>
-	  <material>Gazebo/Blue</material>
 	  <plugin name='altimeter_plugin' filename='libplugin_altimeter.so'>
 		<bodyName>altimeter</bodyName>
-		<robotNamespace>/viman</robotNamespace>
 		<frameId>altimeter</frameId>
-		<altimeterTopicName>/height</altimeterTopicName>
-		<elevation>0</elevation>
+		<altimeterTopicName>/viman/height</altimeterTopicName>
+		<noise>0.01</noise>
 	  </plugin>
   </gazebo>

Commit message: added imu; yaw PID

File: viman_visualize/urdf/viman.xacro (robot description, xacro)
@@ -6,4 +6,6 @@
   <xacro:property name="altimeter_origin_offset" value="0 0 0.015"/>
   <xacro:property name="altimeter_dimensions" value="0.005 0.005 0.002"/>
+  <xacro:property name="imu_origin_offset" value="0 0 0.017"/>
+  <xacro:property name="imu_dimensions" value="0.005 0.005 0.002"/>
   <!-- Macro to define propeller links -->
   <!-- Input parameters: propeller ID, pose of the joint, xyz of CoM -->
@@ -104,4 +106,84 @@
   <xacro:propeller_link id="3" com="-2.7756E-17 -0.00027271 0" xyz="0.085003 0.084703 0.0335" rpy="1.5708 0 1.1739"/>
   <xacro:propeller_link id="4" com="2.7756E-17 -0.00027271 2.7756E-17" xyz="-0.084703 0.085003 0.0335" rpy="1.5708 0 2.5345"/>
+  <link name="altimeter">
+    <collision>
+      <origin xyz="0 0 0" rpy="0 0 0"/>
+      <geometry>
+		<box size="${altimeter_dimensions}"/>
+      </geometry>
+    </collision>
+    <visual>
+      <origin xyz="0 0 0" rpy="0 0 0"/>
+      <geometry>
+    <box size="${altimeter_dimensions}"/>
+      </geometry>
+      <material name="blue"/>
+    </visual>
+    <inertial>
+      <mass value="1e-5" />
+      <origin xyz="0 0 0" rpy="0 0 0"/>
+      <inertia ixx="1e-6" ixy="0" ixz="0" iyy="1e-6" iyz="0" izz="1e-6" />
+    </inertial>
+  </link>
+  <joint name="altimeter_joint" type="fixed">
+    <origin xyz="${altimeter_origin_offset}" rpy="0 0 0"/>
+    <parent link="base_link"/>
+    <child link="altimeter"/>
+  </joint>
+  <gazebo reference="altimeter">
+	<material>Gazebo/SkyBlue</material>
+  </gazebo>
+  <link name="camera">
+    <collision>
+      <origin xyz="0 0 0" rpy="0 0 0"/>
+      <geometry>
+		<box size="${camera_dimensions}"/>
+      </geometry>
+    </collision>
+    <visual>
+      <origin xyz="0 0 0" rpy="0 0 0"/>
+      <geometry>
+    <box size="${camera_dimensions}"/>
+      </geometry>
+      <material name="red"/>
+    </visual>
+    <inertial>
+      <mass value="1e-5" />
+      <origin xyz="0 0 0" rpy="0 0 0"/>
+      <inertia ixx="1e-6" ixy="0" ixz="0" iyy="1e-6" iyz="0" izz="1e-6" />
+    </inertial>
+  </link>
+  <joint name="camera_joint" type="fixed">
+    <origin xyz="${cam_origin_offset}" rpy="0 0 -1.5708"/>
+    <parent link="base_link"/>
+    <child link="camera"/>
+  </joint>
+  <link name="imu_link">
+    <collision>
+      <origin xyz="0 0 0" rpy="0 0 0"/>
+      <geometry>
+		<box size="${imu_dimensions}"/>
+      </geometry>
+    </collision>
+    <visual>
+      <origin xyz="0 0 0" rpy="0 0 0"/>
+      <geometry>
+		<box size="${imu_dimensions}"/>
+      </geometry>
+    </visual>
+    <inertial>
+      <mass value="1e-5" />
+      <origin xyz="0 0 0" rpy="0 0 0"/>
+      <inertia ixx="1e-6" ixy="0" ixz="0" iyy="1e-6" iyz="0" izz="1e-6" />
+    </inertial>
+  </link>
+  <joint name="imu_joint" type="fixed">
+    <origin xyz="${imu_origin_offset}" rpy="0 0 0"/>
+    <parent link="base_link"/>
+    <child link="imu_link"/>
+  </joint>
+  <gazebo reference="imu_link">
+	<material>Gazebo/Purple</material>
+  </gazebo>
   <!-- Flight plugin -->
   <gazebo>
@@ -134,30 +216,5 @@
     </plugin>
   </gazebo>
-  <link name="camera">
-    <collision>
-      <origin xyz="0 0 0" rpy="0 0 0"/>
-      <geometry>
-		<box size="${camera_dimensions}"/>
-      </geometry>
-    </collision>
-    <visual>
-      <origin xyz="0 0 0" rpy="0 0 0"/>
-      <geometry>
-    <box size="${camera_dimensions}"/>
-      </geometry>
-      <material name="red"/>
-    </visual>
-    <inertial>
-      <mass value="1e-5" />
-      <origin xyz="0 0 0" rpy="0 0 0"/>
-      <inertia ixx="1e-6" ixy="0" ixz="0" iyy="1e-6" iyz="0" izz="1e-6" />
-    </inertial>
-  </link>
-  <joint name="camera_joint" type="fixed">
-    <origin xyz="${cam_origin_offset}" rpy="0 0 -1.5708"/>
-    <parent link="base_link"/>
-    <child link="camera"/>
-  </joint>
-  <!-- Camera: Plugin -->
+  <!-- Camera: plugin -->
   <gazebo reference="camera">
 	<material>Gazebo/Red</material>
@@ -200,32 +257,4 @@
     </sensor>
   </gazebo>
-  <link name="altimeter">
-    <collision>
-      <origin xyz="0 0 0" rpy="0 0 0"/>
-      <geometry>
-		<box size="${altimeter_dimensions}"/>
-      </geometry>
-    </collision>
-    <visual>
-      <origin xyz="0 0 0" rpy="0 0 0"/>
-      <geometry>
-    <box size="${altimeter_dimensions}"/>
-      </geometry>
-      <material name="blue"/>
-    </visual>
-    <inertial>
-      <mass value="1e-5" />
-      <origin xyz="0 0 0" rpy="0 0 0"/>
-      <inertia ixx="1e-6" ixy="0" ixz="0" iyy="1e-6" iyz="0" izz="1e-6" />
-    </inertial>
-  </link>
-  <joint name="altimeter_joint" type="fixed">
-    <origin xyz="${altimeter_origin_offset}" rpy="0 0 0"/>
-    <parent link="base_link"/>
-    <child link="altimeter"/>
-  </joint>
-  <gazebo reference="altimeter">
-	<material>Gazebo/SkyBlue</material>
-  </gazebo>
   <!-- Altimeter plugin -->
   <gazebo>
@@ -237,3 +266,34 @@
 	  </plugin>
   </gazebo>
+  <!-- IMU plugin
+  <gazebo reference="imu_link">
+    <gravity>true</gravity>
+    <sensor name="imu_sensor" type="imu">
+      <always_on>true</always_on>
+      <update_rate>100</update_rate>
+      <visualize>true</visualize>
+      <topic>/viman/imu</topic>
+      <plugin filename="libgazebo_ros_imu_sensor.so" name="imu_plugin">
+        <topicName>imu</topicName>
+        <bodyName>imu_link</bodyName>
+        <updateRateHZ>10.0</updateRateHZ>
+        <gaussianNoise>0.0</gaussianNoise>
+        <xyzOffset>0 0 0</xyzOffset>
+        <rpyOffset>0 0 0</rpyOffset>
+        <frameName>imu_link</frameName>
+        <initialOrientationAsReference>false</initialOrientationAsReference>
+      </plugin>
+      <pose>0 0 0 0 0 0</pose>
+    </sensor>
+  </gazebo>-->
+  <gazebo>
+    <plugin name="imu_plugin" filename="libgazebo_ros_imu.so">
+      <alwaysOn>true</alwaysOn>
+      <bodyName>imu_link</bodyName>
+      <topicName>/viman/imu</topicName>
+      <serviceName>imu_service</serviceName>
+      <gaussianNoise>0.0</gaussianNoise>
+      <updateRate>20.0</updateRate>
+    </plugin>
+  </gazebo>
 </robot>

Commit message: added z linear only props

File: viman_visualize/urdf/viman.xacro (robot description, xacro)
@@ -51,5 +51,5 @@
         </link>
         <joint name="propeller_${id}_joint" type="fixed">
-            <parent link="base_link"/>
+            <parent link="viman_base_link"/>
             <child link="propeller_${id}"/>
             <origin rpy="${rpy}" xyz="${xyz}"/>
@@ -60,5 +60,5 @@
 		</gazebo>
   </xacro:macro>
-  <link name="base_link">
+  <link name="viman_base_link">
     <inertial>
       <origin
@@ -99,5 +99,5 @@
     </collision>
   </link>
-  <gazebo reference="base_link">
+  <gazebo reference="viman_base_link">
 	<material>Gazebo/Yellow</material>
   </gazebo>
@@ -128,5 +128,5 @@
   <joint name="altimeter_joint" type="fixed">
     <origin xyz="${altimeter_origin_offset}" rpy="0 0 0"/>
-    <parent link="base_link"/>
+    <parent link="viman_base_link"/>
     <child link="altimeter"/>
   </joint>
@@ -156,5 +156,5 @@
   <joint name="camera_joint" type="fixed">
     <origin xyz="${cam_origin_offset}" rpy="0 0 -1.5708"/>
-    <parent link="base_link"/>
+    <parent link="viman_base_link"/>
     <child link="camera"/>
   </joint>
@@ -180,5 +180,5 @@
   <joint name="imu_joint" type="fixed">
     <origin xyz="${imu_origin_offset}" rpy="0 0 0"/>
-    <parent link="base_link"/>
+    <parent link="viman_base_link"/>
     <child link="imu_link"/>
   </joint>
@@ -189,5 +189,5 @@
   <gazebo>
     <plugin name='viman_flight' filename='libplugin_viman_flight.so'>
-        <bodyName>base_link</bodyName>
+        <bodyName>viman_base_link</bodyName>
         <imuTopic>/viman/imu</imuTopic>
         <rollpitchProportionalGain>10.0</rollpitchProportionalGain>

Commit message: Added Down cam

File: viman_visualize/urdf/viman.xacro (robot description, xacro)
@@ -134,16 +134,16 @@
 	<material>Gazebo/SkyBlue</material>
   </gazebo>
-  <link name="camera">
-    <collision>
-      <origin xyz="0 0 0" rpy="0 0 0"/>
-      <geometry>
-		<box size="${camera_dimensions}"/>
-      </geometry>
-    </collision>
-    <visual>
+  <link name="camera-front">
+    <collision>
       <origin xyz="0 0 0" rpy="0 0 0"/>
       <geometry>
     <box size="${camera_dimensions}"/>
       </geometry>
+    </collision>
+    <visual>
+      <origin xyz="0 0 0" rpy="0 0 0"/>
+      <geometry>
+    <box size="${camera_dimensions}"/>
+      </geometry>
       <material name="red"/>
     </visual>
@@ -154,8 +154,33 @@
     </inertial>
   </link>
-  <joint name="camera_joint" type="fixed">
+  <joint name="camera_joint_frnt" type="fixed">
     <origin xyz="${cam_origin_offset}" rpy="0 0 -1.5708"/>
     <parent link="viman_base_link"/>
-    <child link="camera"/>
+    <child link="camera-front"/>
+  </joint>
+  <link name="camera-down">
+    <collision>
+      <origin xyz="0 0 0" rpy="0 0 0"/>
+      <geometry>
+		<box size="${camera_dimensions}"/>
+      </geometry>
+    </collision>
+    <visual>
+      <origin xyz="0 0 0" rpy="0 0 0"/>
+      <geometry>
+    <box size="${camera_dimensions}"/>
+      </geometry>
+      <material name="red"/>
+    </visual>
+    <inertial>
+      <mass value="1e-5" />
+      <origin xyz="0 0 0" rpy="0 0 0"/>
+      <inertia ixx="1e-6" ixy="0" ixz="0" iyy="1e-6" iyz="0" izz="1e-6" />
+    </inertial>
+  </link>
+  <joint name="camera_joint_down" type="fixed">
+    <origin xyz="0 0 -0.001" rpy="0 1 0"/>
+    <parent link="viman_base_link"/>
+    <child link="camera-down"/>
   </joint>
   <link name="imu_link">
@@ -217,9 +242,45 @@
   </gazebo>
   <!-- Camera: plugin -->
-  <gazebo reference="camera">
+  <gazebo reference="camera-front">
 	<material>Gazebo/Red</material>
     <sensor type="camera" name="vm_frnt_cam">
       <update_rate>30.0</update_rate>
       <camera name="vm_frnt_cam">
+        <horizontal_fov>1.3</horizontal_fov>
+        <image>
+          <width>640</width>
+          <height>480</height>
+        </image>
+        <clip>
+          <near>0.1</near>
+          <far>30</far>
+        </clip>
+        <noise>
+          <type>gaussian</type>
+          <mean>0.0</mean>
+          <stddev>0.007</stddev>
+        </noise>
+      </camera>
+      <plugin name="camera_controller" filename="libgazebo_ros_camera.so">
+        <alwaysOn>true</alwaysOn>
+        <updateRate>30.0</updateRate>
+        <cameraName>viman/vm_frnt_cam</cameraName>
+        <imageTopicName>image</imageTopicName>
+        <cameraInfoTopicName>vm_frnt_cam_info</cameraInfoTopicName>
+        <frameName>camera_link1</frameName>
+        <hackBaseline>0.07</hackBaseline>
+        <distortionK1>0.01</distortionK1>
+        <distortionK2>0.02</distortionK2>
+        <distortionK3>0.01</distortionK3>
+        <distortionT1>0.03</distortionT1>
+        <distortionT2>0.04</distortionT2>
+      </plugin>
+    </sensor>
+  </gazebo>
+   <gazebo reference="camera-down">
+  <material>Gazebo/Red</material>
+    <sensor type="camera" name="vm_down_cam">
+      <update_rate>30.0</update_rate>
+      <camera name="vm_down_cam">
         <horizontal_fov>1.3</horizontal_fov>
         <image>
